Commit message: update head-to-camera transform from manual extrinsic calibration

File: nextagea_description/urdf/NextageAOpen_gazebo_intel_realsense.urdf.xacro (robot description, xacro)
@@ -135,5 +135,5 @@
   <!-- Attach the RealSense D435 -->
   <joint name="d435_mount_joint" type="fixed">
-      <origin xyz="0 0 0.165" rpy="0 0.325 0"/>
+      <origin xyz="0 0 0.1448322" rpy="0 0.24902114520034205 0"/>
       <parent link="HEAD_JOINT1_Link"/>
       <child link="d435_Mount_Link"/>
