Commit message: RealSense Head Mount URDF Inclusion (#20)
* [nextagea_gazebo] Set Gazebo launch URDF default behaviour and create launch file for realsense

* [nextagea_description] Add Realsense files and resources

* [nextagea_description] Initial positioning of the Realsense

* [nextagea_description] Further refinements to Realsense position

* [nextagea_description] Add 3D sensor map

* [nextagea_description] Add inertial term to realsense mount

File: nextagea_description/urdf/common.xacro (robot description, xacro)
@@ -39,3 +39,6 @@
         </xacro:macro>
     </xacro:if>
+    <xacro:macro name="sphere_inertia_def" params="radius mass">
+        <inertia ixx="${2/5*mass*radius*radius}" ixy="0" ixz="0" iyy="${2/5*mass*radius*radius}" iyz="0" izz="${2/5*mass*radius*radius}"/>
+    </xacro:macro>
 </robot>

Commit message: Fixed formatting

File: nextagea_description/urdf/common.xacro (robot description, xacro)
@@ -29,11 +29,11 @@
         <xacro:macro name="gazebo_nx_link" params="name color">
             <gazebo reference="gazebo_${name}">
-            <material>Gazebo/${color}</material>
-            <mu1 value="1.0" />
-            <mu2 value="1.0" />
-            <kp  value="1000000.0" />
-            <kd  value="100.0" />
-            <maxVel  value="100.0" />
-            <minDepth  value="0.0" />
+                <material>Gazebo/${color}</material>
+                <mu1 value="1.0" />
+                <mu2 value="1.0" />
+                <kp  value="1000000.0" />
+                <kd  value="100.0" />
+                <maxVel  value="100.0" />
+                <minDepth  value="0.0" />
             </gazebo>
         </xacro:macro>
