Commit message: Fixed integration, plotting, tuned gains (#19)

File: nextagea_description/urdf/NextageA_robot.xacro (robot description, xacro)
@@ -2,4 +2,6 @@
 <robot xmlns:xacro="http://ros.org/wiki/xacro">
   <xacro:include filename="$(find nextagea_description)/urdf/common.xacro" />
+  <xacro:property name="namespace" default="/nextagea/" />
+  <xacro:property name="nextagea_gazebo_ros_control" default="true" />
   <xacro:gazebo_nx_link name="WAIST" color="Black" />
   <link name="WAIST">
@@ -612,7 +614,11 @@
   </joint>
   <!-- Gazebo plugin for ROS Control -->
-  <gazebo>
-    <plugin name="gazebo_ros_control" filename="libgazebo_ros_control.so" />
-  </gazebo>
+  <xacro:if value="${nextagea_gazebo_ros_control}">
+    <gazebo>
+      <plugin name="gazebo_ros_control" filename="libgazebo_ros_control.so">
+        <robotNamespace>${namespace}</robotNamespace>
+      </plugin>
+    </gazebo>
+  </xacro:if>
   <!-- Gazebo-Specific Link Properties -->
   <gazebo reference="CHEST_JOINT0">

Commit message: [nextagea_description] Decreased Joint4 lower limit for safety

File: nextagea_description/urdf/NextageA_robot.xacro (robot description, xacro)
@@ -523,5 +523,5 @@
     <origin xyz="0.1495 0 0" rpy="0 0 0"/>
     <axis xyz="0 1 0"/>
-    <limit lower="-3.57792" upper="1.134464" effort="150" velocity="1.0"/>
+    <limit lower="-2.9" upper="1.134464" effort="150" velocity="1.0"/>
     <dynamics damping="0.5" friction="0.5"/>
   </joint>
@@ -577,5 +577,5 @@
     <origin xyz="0.1495 0 0" rpy="0 0 0"/>
     <axis xyz="0 1 0"/>
-    <limit lower="-3.5779" upper="1.134464" effort="150" velocity="1.0"/>
+    <limit lower="-2.9" upper="1.134464" effort="150" velocity="1.0"/>
     <dynamics damping="0.5" friction="0.5"/>
   </joint>

Commit message: set joint velocity limits in URDF

File: nextagea_description/urdf/NextageA_robot.xacro (robot description, xacro)
@@ -462,5 +462,5 @@
     <origin xyz="0 0 0.267" rpy="0 0 0"/>
     <axis xyz="0 0 1"/>
-    <limit lower="-3.14159" upper="3.14159" effort="100" velocity="1.0"/>
+    <limit lower="-3.14159" upper="3.14159" effort="100" velocity="2.513274"/>
     <dynamics damping="0.2" friction="0"/>
   </joint>
@@ -471,5 +471,5 @@
     <origin xyz="0 0 0.302" rpy="0 0 0"/>
     <axis xyz="0 0 1"/>
-    <limit lower="-1.22173" upper="1.22173" effort="100" velocity="1.0"/>
+    <limit lower="-1.22173" upper="1.22173" effort="100" velocity="6.684611"/>
   </joint>
   <xacro:transmission_nx_joint name="HEAD_JOINT1" />
@@ -479,5 +479,5 @@
     <origin xyz="0 0 0.08" rpy="0 0 0"/>
     <axis xyz="0 1 0"/>
-    <limit lower="-0.401425" upper="1.308997" effort="100" velocity="1.0"/>
+    <limit lower="-0.401425" upper="1.308997" effort="100" velocity="6.684611"/>
   </joint>
   <xacro:transmission_nx_joint name="LARM_JOINT0" />
@@ -487,5 +487,5 @@
     <origin xyz="0.04 0.135 0.1015" rpy="0 0 0"/>
     <axis xyz="0 0 1"/>
-    <limit lower="-1.5707963" upper="1.5707963" effort="150" velocity="1.0"/>
+    <limit lower="-1.5707963" upper="1.5707963" effort="150" velocity="3.892084"/>
     <dynamics damping="0.5" friction="0.5"/>
   </joint>
@@ -496,5 +496,5 @@
     <origin xyz="0 0 0.066" rpy="0 0 0"/>
     <axis xyz="0 1 0"/>
-    <limit lower="-2.44346" upper="1.0471975" effort="150" velocity="1.0"/>
+    <limit lower="-2.44346" upper="1.0471975" effort="150" velocity="2.426008"/>
     <dynamics damping="0.5" friction="0.5"/>
   </joint>
@@ -505,5 +505,5 @@
     <origin xyz="0 0.095 -0.25" rpy="0 0 0"/>
     <axis xyz="0 1 0"/>
-    <limit lower="-1.22173" upper="1.5707963" effort="150" velocity="1.0"/>
+    <limit lower="-1.22173" upper="1.5707963" effort="150" velocity="3.630285"/>
     <dynamics damping="0.5" friction="0.5"/>
   </joint>
@@ -514,5 +514,5 @@
     <origin xyz="0.1805 0 -0.03" rpy="0 0 0"/>
     <axis xyz="1 0 0"/>
-    <limit lower="-3.1415926" upper="1.7453292" effort="150" velocity="1.0"/>
+    <limit lower="-3.1415926" upper="1.7453292" effort="150" velocity="6.352998"/>
     <dynamics damping="0.5" friction="0.5"/>
   </joint>
@@ -523,5 +523,5 @@
     <origin xyz="0.1495 0 0" rpy="0 0 0"/>
     <axis xyz="0 1 0"/>
-    <limit lower="-2.9" upper="1.134464" effort="150" velocity="1.0"/>
+    <limit lower="-2.9" upper="1.134464" effort="150" velocity="6.352998"/>
     <dynamics damping="0.5" friction="0.5"/>
   </joint>
@@ -532,5 +532,5 @@
     <origin xyz="0 0 -0.1335" rpy="0 0 0"/>
     <axis xyz="0 0 1"/>
-    <limit lower="-2.7123889" upper="2.7123889" effort="150" velocity="1.0"/>
+    <limit lower="-2.7123889" upper="2.7123889" effort="150" velocity="6.352998"/>
     <dynamics damping="0.5" friction="0.5"/>
   </joint>
@@ -541,5 +541,5 @@
     <origin xyz="0.04 -0.135 0.1015" rpy="0 0 0"/>
     <axis xyz="0 0 1"/>
-    <limit lower="-1.570796" upper="1.570796" effort="150" velocity="1.0"/>
+    <limit lower="-1.570796" upper="1.570796" effort="150" velocity="3.892084"/>
     <dynamics damping="0.5" friction="0.5"/>
   </joint>
@@ -550,5 +550,5 @@
     <origin xyz="0 0 0.066" rpy="0 0 0"/>
     <axis xyz="0 1 0"/>
-    <limit lower="-2.44346" upper="1.047197" effort="150" velocity="1.0"/>
+    <limit lower="-2.44346" upper="1.047197" effort="150" velocity="2.426008"/>
     <dynamics damping="0.5" friction="0.5"/>
   </joint>
@@ -559,5 +559,5 @@
     <origin xyz="0 -0.095 -0.25" rpy="0 0 0"/>
     <axis xyz="0 1 0"/>
-    <limit lower="-1.22173" upper="1.570796" effort="150" velocity="1.0"/>
+    <limit lower="-1.22173" upper="1.570796" effort="150" velocity="3.630285"/>
     <dynamics damping="0.5" friction="0.5"/>
   </joint>
@@ -568,5 +568,5 @@
     <origin xyz="0.1805 0 -0.03" rpy="0 0 0"/>
     <axis xyz="1 0 0"/>
-    <limit lower="-1.74532" upper="3.141592" effort="150" velocity="1.0"/>
+    <limit lower="-1.74532" upper="3.141592" effort="150" velocity="6.352998"/>
     <dynamics damping="0.5" friction="0.5"/>
   </joint>
@@ -577,5 +577,5 @@
     <origin xyz="0.1495 0 0" rpy="0 0 0"/>
     <axis xyz="0 1 0"/>
-    <limit lower="-2.9" upper="1.134464" effort="150" velocity="1.0"/>
+    <limit lower="-2.9" upper="1.134464" effort="150" velocity="6.352998"/>
     <dynamics damping="0.5" friction="0.5"/>
   </joint>
@@ -586,5 +586,5 @@
     <origin xyz="0 0 -0.1335" rpy="0 0 0"/>
     <axis xyz="0 0 1"/>
-    <limit lower="-2.712388" upper="2.712388" effort="150" velocity="1.0"/>
+    <limit lower="-2.712388" upper="2.712388" effort="150" velocity="6.352998"/>
     <dynamics damping="0.5" friction="0.5"/>
   </joint>

Commit message: Added collision shapes for cables around the wrist

File: nextagea_description/urdf/NextageA_robot.xacro (robot description, xacro)
@@ -643,3 +643,41 @@
     <implicitSpringDamper>1</implicitSpringDamper>
   </gazebo>
+  <joint name="LARM_JOINT4_Link_cables_joint" type="fixed">
+    <parent link="LARM_JOINT4_Link"/>
+    <child link="LARM_JOINT4_Link_cables"/>
+    <origin xyz="0 0 0" rpy="0 0 0"/>
+    <axis xyz="0 0 1"/>
+  </joint>
+  <joint name="RARM_JOINT4_Link_cables_joint" type="fixed">
+    <parent link="RARM_JOINT4_Link"/>
+    <child link="RARM_JOINT4_Link_cables"/>
+    <origin xyz="0 0 0" rpy="0 0 0"/>
+    <axis xyz="0 0 1"/>
+  </joint>
+  <link name="LARM_JOINT4_Link_cables">
+    <inertial>
+      <mass value="0.01" />
+      <origin xyz="0 0 0" rpy="0 0 0"/>
+      <xacro:nxa_box_inertia_def x="0.016" y="0.006" z="0.012" mass="0.01"/>
+    </inertial>
+    <collision>
+      <origin xyz="0 0.08 -0.1" rpy="0 0 0"/>
+      <geometry>
+        <sphere radius="0.1"/>
+      </geometry>
+    </collision>
+  </link>
+  <link name="RARM_JOINT4_Link_cables">
+    <inertial>
+      <mass value="0.01" />
+      <origin xyz="0 0 0" rpy="0 0 0"/>
+      <xacro:nxa_box_inertia_def x="0.016" y="0.006" z="0.012" mass="0.01"/>
+    </inertial>
+    <collision>
+      <origin xyz="0 -0.08 -0.1" rpy="0 0 0"/>
+      <geometry>
+        <sphere radius="0.1"/>
+      </geometry>
+    </collision>
+  </link>
 </robot>

Commit message: Fix too conservative joint position limit

File: nextagea_description/urdf/NextageA_robot.xacro (robot description, xacro)
@@ -523,5 +523,5 @@
     <origin xyz="0.1495 0 0" rpy="0 0 0"/>
     <axis xyz="0 1 0"/>
-    <limit lower="-2.9" upper="1.134464" effort="150" velocity="6.352998"/>
+    <limit lower="-3.4" upper="1.134464" effort="150" velocity="6.352998"/>
     <dynamics damping="0.5" friction="0.5"/>
   </joint>
@@ -577,5 +577,5 @@
     <origin xyz="0.1495 0 0" rpy="0 0 0"/>
     <axis xyz="0 1 0"/>
-    <limit lower="-2.9" upper="1.134464" effort="150" velocity="6.352998"/>
+    <limit lower="-3.4" upper="1.134464" effort="150" velocity="6.352998"/>
     <dynamics damping="0.5" friction="0.5"/>
   </joint>
