Commit message: URDF fixes (#26)
* set world frame to ground plane

* use original RealSense xacro file

* split hand-camera links

* fix whitespace

* split camera links out of main robot xacro

* define and activate FT-sensor link

* move hand-camera frame definitions to main robot file

File: nextagea_description/urdf/NextageAOpen.urdf.xacro (robot description, xacro)
@@ -18,3 +18,103 @@
   <xacro:include filename="$(find nextagea_description)/urdf/NextageA_base.xacro" />
   <xacro:include filename="$(find nextagea_description)/urdf/NextageA_robot.xacro" />
+  <xacro:include filename="$(find nextagea_description)/urdf/nxao_gz_camera.xacro" />
+  <xacro:arg name="use_hand_cameras" default="false"/>
+  <xacro:arg name="use_ft_sensors" default="false"/>
+  <xacro:macro name="nxao_camera" params="prefix parent">
+    <xacro:if value="${prefix == 'L'}">
+      <xacro:property name="m" value="+1" />
+    </xacro:if>
+    <xacro:if value="${prefix == 'R'}">
+      <xacro:property name="m" value="-1" />
+    </xacro:if>
+    <xacro:gazebo_nx_link name="${prefix}ARM_camera_Link" color="Black" />
+    <link name="${prefix}ARM_camera_Link">
+      <visual>
+        <origin xyz="0 0 0" rpy="0 0 0"/>
+        <geometry>
+          <mesh filename="package://nextagea_description/urdf/meshes/${prefix}_CAM.dae"/>
+        </geometry>
+      </visual>
+      <collision>
+        <origin xyz="0 0 -0.025" rpy="0 0 0"/>
+        <geometry>
+          <cylinder length="0.05" radius="0.037"/>
+        </geometry>
+      </collision>
+      <collision>
+        <origin xyz="0.0525 ${m * 0.029} -0.02" rpy="0 0 0"/>
+        <geometry>
+          <box size="0.057 0.106 0.042"/>
+        </geometry>
+      </collision>
+      <inertial>
+        <mass value="1.05156" />
+        <origin xyz="0.0 0.0 -0.08" rpy="0 -0 0"/>
+        <inertia ixx="0.00194072" ixy="${m * 1.1e-07}" ixz="-0.00042482" iyy="0.00209392" iyz="${m * 1.2e-07}" izz="0.00035788"/>
+      </inertial>
+    </link>
+    <joint name="${prefix}ARM_JOINT6" type="fixed">
+      <parent link="${parent}"/>
+      <child link="${prefix}ARM_camera_Link"/>
+      <origin xyz="0 0 0" rpy="0 0 0"/>
+      <axis xyz="0 0 1"/>
+    </joint>
+    <xacro:camera_joint_link_gzplugin
+      camera_name="CAMERA_HAND_${prefix}" link_parent="${parent}"
+      jnt_displacement_x="${jnt_hand_camera_displacement_x}"
+      jnt_displacement_y="${m * jnt_hand_camera_displacement_y}"
+      jnt_displacement_z="${jnt_hand_camera_displacement_z}"
+      jnt_rotation_x="0" jnt_rotation_y="${jnt_hand_camera_rot_y}" jnt_rotation_z="0"
+      link_displacement_x="0.0325" link_displacement_y="0" link_displacement_z="0"
+      link_rotation_x="0" link_rotation_y="${M_PI/2}" link_rotation_z="-${link_hand_camera_rot_z}" />
+  </xacro:macro>
+  <xacro:macro name="nxao_ft_sensor" params="prefix parent">
+    <xacro:if value="${prefix == 'L'}">
+      <xacro:property name="m" value="+1" />
+    </xacro:if>
+    <xacro:if value="${prefix == 'R'}">
+      <xacro:property name="m" value="-1" />
+    </xacro:if>
+    <xacro:gazebo_nx_link name="${prefix}ARM_ft_Link" color="LightGrey" />
+    <link name="${prefix}ARM_ft_Link">
+      <visual>
+        <origin xyz="0 0 0.0185" rpy="0 0 0"/>
+        <geometry>
+          <cylinder length="0.037" radius="0.035"/>
+        </geometry>
+        <material name="LightGrey">
+          <color rgba="0.6 0.6 0.6 1.0"/>
+        </material>
+      </visual>
+      <collision>
+        <origin xyz="0 0 0.0185" rpy="0 0 0"/>
+        <geometry>
+          <cylinder length="0.037" radius="0.04"/>
+        </geometry>
+      </collision>
+      <!-- TODO: The inertial values are copied from ARM_JOINT5_Link. Replace with proper values. -->
+      <inertial>
+        <mass value="1.05156" />
+        <origin xyz="0.0 0.0 -0.08" rpy="0 -0 0"/>
+        <inertia ixx="0.00194072" ixy="1.1e-07" ixz="-0.00042482" iyy="0.00209392" iyz="1.2e-07" izz="0.00035788"/>
+      </inertial>
+    </link>
+    <joint name="${prefix}ARM_ft_joint" type="fixed">
+      <parent link="${parent}"/>
+      <child link="${prefix}ARM_ft_Link"/>
+      <origin xyz="0 0 -0.037" rpy="0 0 0"/>
+      <axis xyz="0 0 1"/>
+    </joint>
+  </xacro:macro>
+  <xacro:property name="arm_tip" value="ARM_JOINT5_Link" />
+  <xacro:if value="$(arg use_ft_sensors)">
+    <xacro:nxao_ft_sensor prefix="L" parent="L${arm_tip}" />
+    <xacro:nxao_ft_sensor prefix="R" parent="R${arm_tip}" />
+    <xacro:property name="arm_tip" value="ARM_ft_Link" />
+  </xacro:if>
+  <xacro:if value="$(arg use_hand_cameras)">
+    <xacro:nxao_camera prefix="L" parent="L${arm_tip}" />
+    <xacro:nxao_camera prefix="R" parent="R${arm_tip}" />
+    <xacro:property name="arm_tip" value="ARM_camera_Link" />
+  </xacro:if>
 </robot>

File: nextagea_description/urdf/NextageAOpen_gazebo.urdf.xacro (robot description, xacro)
@@ -5,5 +5,4 @@
   <xacro:include filename="$(find nextagea_description)/urdf/common.xacro" />
   <xacro:include filename="$(find nextagea_description)/urdf/NextageAOpen.urdf.xacro" />
-  <xacro:include filename="$(find nextagea_description)/urdf/nxao_gz_camera.xacro" />
   <!-- Used for fixing robot to Gazebo 'base_link' -->
   <xacro:if value="${fixed_base}">
@@ -12,5 +11,5 @@
       <parent link="world"/>
       <child link="base_link"/>
-      <origin xyz="0 0 -0.15" rpy="0 0 0"/>
+      <origin xyz="0 0 0.85" rpy="0 0 0"/>
     </joint>
   </xacro:if>

File: nextagea_description/urdf/NextageAOpen_gazebo_intel_realsense.urdf.xacro (robot description, xacro)
@@ -3,6 +3,134 @@
        xmlns:xacro="http://www.ros.org/wiki/xacro">
   <xacro:property name="fixed_base" value="True" />
+  <xacro:property name="ft_sensors" value="True" />
+  <xacro:property name="hand_camera" value="True" />
   <xacro:include filename="$(find nextagea_description)/urdf/NextageAOpen_gazebo.urdf.xacro" />
-  <xacro:include filename="$(find nextagea_description)/urdf/accessories/d435.urdf.xacro"/>
+  <xacro:include filename="$(find realsense2_description)/urdf/_d435.urdf.xacro"/>
+  <xacro:macro name="sensor_d435_gz" params="name">
+    <gazebo reference="${name}_color_frame">
+      <sensor name="color" type="camera">
+        <pose frame="">0 0 0 0 0 0</pose>
+        <camera name="__default__">
+          <horizontal_fov>1.5009831567151233</horizontal_fov>
+          <image>
+            <width>640</width>
+            <height>480</height>
+            <format>RGB_INT8</format>
+          </image>
+          <clip>
+            <near>0.1</near>
+            <far>100</far>
+          </clip>
+          <noise>
+            <type>gaussian</type>
+            <mean>0.0</mean>
+            <stddev>0.007</stddev>
+          </noise>
+        </camera>
+        <always_on>1</always_on>
+        <update_rate>30</update_rate>
+        <visualize>1</visualize>
+      </sensor>
+    </gazebo>
+    <gazebo reference="${name}_infra1_frame">
+      <sensor name="ired1" type="camera">
+        <pose frame="">0 0 0 0 0 0</pose>
+        <camera name="__default__">
+          <horizontal_fov>1.5009831567151233</horizontal_fov>
+          <image>
+            <width>640</width>
+            <height>480</height>
+            <format>L_INT8</format>
+          </image>
+          <clip>
+            <near>0.1</near>
+            <far>100</far>
+          </clip>
+          <noise>
+            <type>gaussian</type>
+            <mean>0.0</mean>
+            <stddev>0.007</stddev>
+          </noise>
+        </camera>
+        <always_on>1</always_on>
+        <update_rate>30</update_rate>
+        <visualize>0</visualize>
+      </sensor>
+    </gazebo>
+    <gazebo reference="${name}_infra2_frame">
+      <sensor name="ired2" type="camera">
+        <pose frame="">0 0 0 0 0 0</pose>
+        <camera name="__default__">
+          <horizontal_fov>1.5009831567151233</horizontal_fov>
+          <image>
+            <width>640</width>
+            <height>480</height>
+            <format>L_INT8</format>
+          </image>
+          <clip>
+            <near>0.1</near>
+            <far>100</far>
+          </clip>
+          <noise>
+            <type>gaussian</type>
+            <mean>0.0</mean>
+            <stddev>0.007</stddev>
+          </noise>
+        </camera>
+        <always_on>1</always_on>
+        <update_rate>30</update_rate>
+        <visualize>0</visualize>
+      </sensor>
+    </gazebo>
+    <gazebo reference="${name}_depth_frame">
+      <sensor name="depth" type="depth">
+        <pose frame="">0 0 0 0 0 0</pose>
+        <camera name="__default__">
+          <horizontal_fov>1.5009831567151233</horizontal_fov>
+          <image>
+            <width>640</width>
+            <height>480</height>
+          </image>
+          <clip>
+            <near>0.1</near>
+            <far>100</far>
+          </clip>
+          <noise>
+            <type>gaussian</type>
+            <mean>0.0</mean>
+            <stddev>0.007</stddev>
+          </noise>
+        </camera>
+        <always_on>1</always_on>
+        <update_rate>30</update_rate>
+        <visualize>0</visualize>
+      </sensor>
+    </gazebo>
+    <gazebo>
+      <plugin name="${name}" filename="librealsense_gazebo_plugin.so">
+        <depthUpdateRate>30</depthUpdateRate>
+        <colorUpdateRate>30</colorUpdateRate>
+        <infraredUpdateRate>30</infraredUpdateRate>
+        <depthTopicName>depth/image_raw</depthTopicName>
+        <depthCameraInfoTopicName>depth/camera_info</depthCameraInfoTopicName>
+        <colorTopicName>color/image_raw</colorTopicName>
+        <colorCameraInfoTopicName>color/camera_info</colorCameraInfoTopicName>
+        <infrared1TopicName>infrared/image_raw</infrared1TopicName>
+        <infrared1CameraInfoTopicName>infrared/camera_info</infrared1CameraInfoTopicName>
+        <infrared2TopicName>infrared2/image_raw</infrared2TopicName>
+        <infrared2CameraInfoTopicName>infrared2/camera_info</infrared2CameraInfoTopicName>
+        <colorOpticalframeName>camera_color_optical_frame</colorOpticalframeName>
+        <depthOpticalframeName>camera_depth_optical_frame</depthOpticalframeName>
+        <infrared1OpticalframeName>camera_left_ir_optical_frame</infrared1OpticalframeName>
+        <infrared2OpticalframeName>camera_right_ir_optical_frame</infrared2OpticalframeName>
+        <rangeMinDepth>0.1</rangeMinDepth>
+        <rangeMaxDepth>10</rangeMaxDepth>
+        <pointCloud>1</pointCloud>
+        <pointCloudTopicName>depth/color/points</pointCloudTopicName>
+        <pointCloudCutoff>0.15</pointCloudCutoff>
+        <pointCloudCutoffMax>10</pointCloudCutoffMax>
+      </plugin>
+    </gazebo>
+  </xacro:macro>
   <!-- Attach the RealSense D435 -->
   <joint name="d435_mount_joint" type="fixed">
@@ -18,6 +146,7 @@
     </inertial>
   </link>
-  <xacro:sensor_d435 name="/nextagea/realsense" parent="d435_Mount_Link">
+  <xacro:sensor_d435 name="nextagea_realsense" parent="d435_Mount_Link" use_nominal_extrinsics="true">
       <origin xyz="0 0 0" rpy="0 0 0"/>
   </xacro:sensor_d435>
+  <xacro:sensor_d435_gz name="nextagea_realsense" />
 </robot>

File: nextagea_description/urdf/NextageA_robot.xacro (robot description, xacro)
@@ -276,20 +276,8 @@
       </geometry>
     </visual>
-    <visual>
-      <origin xyz="0 0 0" rpy="0 0 0"/>
-      <geometry>
-	      <mesh filename="package://nextagea_description/urdf/meshes/L_CAM.dae"/>
-      </geometry>
-    </visual>
-    <collision>
-      <origin xyz="0 0 -0.02" rpy="0 0 0"/>
-      <geometry>
-        <cylinder length="0.07" radius="0.037"/>
-      </geometry>
-    </collision>
-    <collision>
-      <origin xyz="0.0525 0.029 -0.02" rpy="0 0 0"/>
-      <geometry>
-        <box size="0.057 0.106 0.042"/>
+    <collision>
+      <origin xyz="0 0 0.0065" rpy="0 0 0"/>
+      <geometry>
+        <cylinder length="0.013" radius="0.037"/>
       </geometry>
     </collision>
@@ -456,20 +444,8 @@
       </geometry>
     </visual>
-    <visual>
-      <origin xyz="0 0 0" rpy="0 0 0"/>
-      <geometry>
-	      <mesh filename="package://nextagea_description/urdf/meshes/R_CAM.dae"/>
-      </geometry>
-    </visual>
-    <collision>
-      <origin xyz="0 0 -0.02" rpy="0 0 0"/>
-      <geometry>
-        <cylinder length="0.07" radius="0.037"/>
-      </geometry>
-    </collision>
-    <collision>
-      <origin xyz="0.0525 -0.029 -0.02" rpy="0 0 0"/>
-      <geometry>
-        <box size="0.057 0.106 0.042"/>
+    <collision>
+      <origin xyz="0 0 0.0065" rpy="0 0 0"/>
+      <geometry>
+        <cylinder length="0.013" radius="0.037"/>
       </geometry>
     </collision>

File: nextagea_description/urdf/nxao_gz_camera.xacro (robot description, xacro)
@@ -100,15 +100,3 @@
 			link_displacement_x="0.0325" link_displacement_y="0" link_displacement_z="0"
 			link_rotation_x="0" link_rotation_y="${M_PI/2}" link_rotation_z="${link_head_camera_rot_z}" />
-	<xacro:camera_joint_link_gzplugin
-			camera_name="CAMERA_HAND_L" link_parent="LARM_JOINT5_Link"
-			jnt_displacement_x="${jnt_hand_camera_displacement_x}" jnt_displacement_y="${jnt_hand_camera_displacement_y}" jnt_displacement_z="${jnt_hand_camera_displacement_z}"
-			jnt_rotation_x="0" jnt_rotation_y="${jnt_hand_camera_rot_y}" jnt_rotation_z="0"
-			link_displacement_x="0.0325" link_displacement_y="0" link_displacement_z="0"
-			link_rotation_x="0" link_rotation_y="${M_PI/2}" link_rotation_z="-${link_hand_camera_rot_z}" />
-	<xacro:camera_joint_link_gzplugin
-			camera_name="CAMERA_HAND_R" link_parent="RARM_JOINT5_Link"
-			jnt_displacement_x="${jnt_hand_camera_displacement_x}" jnt_displacement_y="-${jnt_hand_camera_displacement_y}" jnt_displacement_z="${jnt_hand_camera_displacement_z}"
-			jnt_rotation_x="0" jnt_rotation_y="${jnt_hand_camera_rot_y}" jnt_rotation_z="0"
-			link_displacement_x="0.0325" link_displacement_y="0" link_displacement_z="0"
-			link_rotation_x="0" link_rotation_y="${M_PI/2}" link_rotation_z="-${link_hand_camera_rot_z}" />
 </robot>

Commit message: Fixed FT sensors

File: nextagea_description/urdf/NextageAOpen.urdf.xacro (robot description, xacro)
@@ -72,10 +72,12 @@
     <xacro:if value="${prefix == 'L'}">
       <xacro:property name="m" value="+1" />
+      <xacro:property name="ft_side" value="left" />
     </xacro:if>
     <xacro:if value="${prefix == 'R'}">
       <xacro:property name="m" value="-1" />
+      <xacro:property name="ft_side" value="right" />
     </xacro:if>
     <xacro:gazebo_nx_link name="${prefix}ARM_ft_Link" color="LightGrey" />
-    <link name="${prefix}ARM_ft_Link">
+    <link name="${prefix}ARM_ft_Link_base">
       <visual>
         <origin xyz="0 0 0.0185" rpy="0 0 0"/>
@@ -102,8 +104,50 @@
     <joint name="${prefix}ARM_ft_joint" type="fixed">
       <parent link="${parent}"/>
-      <child link="${prefix}ARM_ft_Link"/>
+      <child link="${prefix}ARM_ft_Link_base"/>
       <origin xyz="0 0 -0.037" rpy="0 0 0"/>
       <axis xyz="0 0 1"/>
     </joint>
+    <link name="${prefix}ARM_ft_Sensor_Link">
+      <inertial>
+        <mass value="0.0001" />
+        <origin xyz="0 0 0" rpy="0 0 0"/>
+        <xacro:nxa_sphere_inertia_def radius="0.0001" mass="0.0001"/>
+      </inertial>
+    </link>
+    <link name="${prefix}ARM_ft_Link">
+      <inertial>
+        <mass value="0.0001" />
+        <origin xyz="0 0 0" rpy="0 0 0"/>
+        <xacro:nxa_sphere_inertia_def radius="0.0001" mass="0.0001"/>
+      </inertial>
+    </link>
+    <joint name="${prefix}ARM_ft_sensor_joint" type="fixed">
+      <parent link="${prefix}ARM_ft_Link_base"/>
+      <child link="${prefix}ARM_ft_Sensor_Link"/>
+      <origin xyz="0 0 0" rpy="0 3.1415 1.57"/>
+      <axis xyz="0 0 1"/>
+    </joint>
+    <joint name="${prefix}ARM_ft_sensor_offset_joint" type="fixed">
+      <parent link="${prefix}ARM_ft_Sensor_Link"/>
+      <child link="${prefix}ARM_ft_Link"/>
+      <origin xyz="0 0 0" rpy="0 3.1415 1.57"/>
+      <axis xyz="0 0 1"/>
+    </joint>
+    <gazebo reference="${prefix}ARM_ft_sensor_joint">
+      <disableFixedJointLumping>true</disableFixedJointLumping>
+      <sensor name="${prefix}ARM_ft_sensor" type="force_torque">
+        <force_torque>
+          <frame>parent</frame>
+          <measure_direction>child_to_parent</measure_direction>
+        </force_torque>
+      </sensor>
+    </gazebo>
+    <gazebo>
+        <plugin name="${prefix}ARM_ft_sensor" filename="libgazebo_ros_ft_sensor.so">
+            <updateRate>500.0</updateRate>
+            <topicName>ft_${ft_side}/data</topicName>
+            <jointName>${prefix}ARM_ft_sensor_joint</jointName>
+        </plugin>
+    </gazebo>
   </xacro:macro>
   <xacro:property name="arm_tip" value="ARM_JOINT5_Link" />

Commit message: move 'fixed_base' macro to main file

File: nextagea_description/urdf/NextageAOpen.urdf.xacro (robot description, xacro)
@@ -19,4 +19,5 @@
   <xacro:include filename="$(find nextagea_description)/urdf/NextageA_robot.xacro" />
   <xacro:include filename="$(find nextagea_description)/urdf/nxao_gz_camera.xacro" />
+  <xacro:arg name="fixed_base" default="true" />
   <xacro:arg name="use_hand_cameras" default="false"/>
   <xacro:arg name="use_ft_sensors" default="false"/>
@@ -152,4 +153,12 @@
   </xacro:macro>
   <xacro:property name="arm_tip" value="ARM_JOINT5_Link" />
+  <xacro:if value="$(arg fixed_base)">
+    <link name="world"/>
+    <joint name="fixed" type="fixed">
+      <parent link="world"/>
+      <child link="base_link"/>
+      <origin xyz="0 0 0.85" rpy="0 0 0"/>
+    </joint>
+  </xacro:if>
   <xacro:if value="$(arg use_ft_sensors)">
     <xacro:nxao_ft_sensor prefix="L" parent="L${arm_tip}" />

File: nextagea_description/urdf/NextageAOpen_gazebo.urdf.xacro (robot description, xacro)
@@ -2,15 +2,5 @@
 <robot name="NextageAOpen"
        xmlns:xacro="http://www.ros.org/wiki/xacro">
-  <xacro:property name="fixed_base" value="True" />
   <xacro:include filename="$(find nextagea_description)/urdf/common.xacro" />
   <xacro:include filename="$(find nextagea_description)/urdf/NextageAOpen.urdf.xacro" />
-  <!-- Used for fixing robot to Gazebo 'base_link' -->
-  <xacro:if value="${fixed_base}">
-    <link name="world"/> -->
-    <joint name="fixed" type="fixed">
-      <parent link="world"/>
-      <child link="base_link"/>
-      <origin xyz="0 0 0.85" rpy="0 0 0"/>
-    </joint>
-  </xacro:if>
 </robot>

Commit message: Make cables optional

File: nextagea_description/urdf/NextageAOpen.urdf.xacro (robot description, xacro)
@@ -22,4 +22,6 @@
   <xacro:arg name="use_hand_cameras" default="false"/>
   <xacro:arg name="use_ft_sensors" default="false"/>
+  <xacro:arg name="use_cables_right" default="true"/>
+  <xacro:arg name="use_cables_left" default="true"/>
   <xacro:macro name="nxao_camera" params="prefix parent">
     <xacro:if value="${prefix == 'L'}">
@@ -171,3 +173,45 @@
     <xacro:property name="arm_tip" value="ARM_camera_Link" />
   </xacro:if>
+  <xacro:if value="$(arg use_cables_left)">
+    <joint name="LARM_JOINT4_Link_cables_joint" type="fixed">
+      <parent link="LARM_JOINT4_Link"/>
+      <child link="LARM_JOINT4_Link_cables"/>
+      <origin xyz="0 0 0" rpy="0 0 0"/>
+      <axis xyz="0 0 1"/>
+    </joint>
+    <link name="LARM_JOINT4_Link_cables">
+      <inertial>
+        <mass value="0.01" />
+        <origin xyz="0 0 0" rpy="0 0 0"/>
+        <xacro:nxa_box_inertia_def x="0.016" y="0.006" z="0.012" mass="0.01"/>
+      </inertial>
+      <collision>
+        <origin xyz="0 0.08 -0.1" rpy="0 0 0"/>
+        <geometry>
+          <sphere radius="0.1"/>
+        </geometry>
+      </collision>
+    </link>
+  </xacro:if>
+  <xacro:if value="$(arg use_cables_right)">
+    <joint name="RARM_JOINT4_Link_cables_joint" type="fixed">
+      <parent link="RARM_JOINT4_Link"/>
+      <child link="RARM_JOINT4_Link_cables"/>
+      <origin xyz="0 0 0" rpy="0 0 0"/>
+      <axis xyz="0 0 1"/>
+    </joint>
+    <link name="RARM_JOINT4_Link_cables">
+      <inertial>
+        <mass value="0.01" />
+        <origin xyz="0 0 0" rpy="0 0 0"/>
+        <xacro:nxa_box_inertia_def x="0.016" y="0.006" z="0.012" mass="0.01"/>
+      </inertial>
+      <collision>
+        <origin xyz="0 -0.08 -0.1" rpy="0 0 0"/>
+        <geometry>
+          <sphere radius="0.1"/>
+        </geometry>
+      </collision>
+    </link>
+  </xacro:if>
 </robot>

File: nextagea_description/urdf/NextageA_robot.xacro (robot description, xacro)
@@ -644,41 +644,3 @@
     <implicitSpringDamper>1</implicitSpringDamper>
   </gazebo>
-  <joint name="LARM_JOINT4_Link_cables_joint" type="fixed">
-    <parent link="LARM_JOINT4_Link"/>
-    <child link="LARM_JOINT4_Link_cables"/>
-    <origin xyz="0 0 0" rpy="0 0 0"/>
-    <axis xyz="0 0 1"/>
-  </joint>
-  <joint name="RARM_JOINT4_Link_cables_joint" type="fixed">
-    <parent link="RARM_JOINT4_Link"/>
-    <child link="RARM_JOINT4_Link_cables"/>
-    <origin xyz="0 0 0" rpy="0 0 0"/>
-    <axis xyz="0 0 1"/>
-  </joint>
-  <link name="LARM_JOINT4_Link_cables">
-    <inertial>
-      <mass value="0.01" />
-      <origin xyz="0 0 0" rpy="0 0 0"/>
-      <xacro:nxa_box_inertia_def x="0.016" y="0.006" z="0.012" mass="0.01"/>
-    </inertial>
-    <collision>
-      <origin xyz="0 0.08 -0.1" rpy="0 0 0"/>
-      <geometry>
-        <sphere radius="0.1"/>
-      </geometry>
-    </collision>
-  </link>
-  <link name="RARM_JOINT4_Link_cables">
-    <inertial>
-      <mass value="0.01" />
-      <origin xyz="0 0 0" rpy="0 0 0"/>
-      <xacro:nxa_box_inertia_def x="0.016" y="0.006" z="0.012" mass="0.01"/>
-    </inertial>
-    <collision>
-      <origin xyz="0 -0.08 -0.1" rpy="0 0 0"/>
-      <geometry>
-        <sphere radius="0.1"/>
-      </geometry>
-    </collision>
-  </link>
 </robot>
