Commit message: added macros to wrap around each object

File: nextagea_description/urdf/base/nextagea_base.xacro (robot description, xacro)
@@ -2,56 +2,58 @@
 <robot xmlns:xacro="http://ros.org/wiki/xacro">
   <xacro:include filename="$(find nextagea_description)/urdf/general/common.xacro" />
-  <!-- Work-around for KDL base-link inertia problem; also adheres to ROS standard-->
-  <link name="base_link"/>
-  <joint name="base_to_dummy" type="fixed">
-    <parent link="base_link"/>
-    <child link="nextage_base"/>
-  </joint>
-  <link name="nextage_base">
-    <visual>
-      <origin xyz="0 0 0" rpy="0 0 0"/>
-      <geometry>
-	      <mesh filename="package://nextagea_description/urdf/meshes/BASE_Link_mesh.dae"/>
-      </geometry>
-    </visual>
-    <collision>
-      <origin xyz="-0.19 0 -0.435" rpy="0 0 0"/>
-      <geometry>
-        <box size="0.585 0.585 0.72"/>
-      </geometry>
-    </collision>
-    <collision>
-      <origin xyz="0.0675 0.2575 -0.82" rpy="0 0 0"/>
-      <geometry>
-        <sphere radius="0.03"/>
-      </geometry>
-    </collision>
-    <collision>
-      <origin xyz="0.0675 -0.2575 -0.82" rpy="0 0 0"/>
-      <geometry>
-        <sphere radius="0.03"/>
-      </geometry>
-    </collision>
-    <collision>
-      <origin xyz="-0.4475 0.2575 -0.82" rpy="0 0 0"/>
-      <geometry>
-        <sphere radius="0.03"/>
-      </geometry>
-    </collision>
-    <collision>
-      <origin xyz="-0.4475 -0.2575 -0.82" rpy="0 0 0"/>
-      <geometry>
-        <sphere radius="0.03"/>
-      </geometry>
-    </collision>
-    <inertial>
-      <mass value="40" />
-      <origin xyz="-0.19 0 -0.435" rpy="0 0 0"/>
-      <xacro:nxa_box_inertia_def x="0.585" y="0.585" z="0.72" mass="40"/>
-    </inertial>
-  </link>
-  <joint name="base_to_waist" type="fixed">
-    <parent link="nextage_base"/>
-    <child link="WAIST"/>
-  </joint>
+  <xacro:macro name="nextagea_base">
+    <!-- Work-around for KDL base-link inertia problem; also adheres to ROS standard-->
+    <link name="base_link"/>
+    <joint name="base_to_dummy" type="fixed">
+      <parent link="base_link"/>
+      <child link="nextage_base"/>
+    </joint>
+    <link name="nextage_base">
+      <visual>
+        <origin xyz="0 0 0" rpy="0 0 0"/>
+        <geometry>
+          <mesh filename="package://nextagea_description/urdf/meshes/BASE_Link_mesh.dae"/>
+        </geometry>
+      </visual>
+      <collision>
+        <origin xyz="-0.19 0 -0.435" rpy="0 0 0"/>
+        <geometry>
+          <box size="0.585 0.585 0.72"/>
+        </geometry>
+      </collision>
+      <collision>
+        <origin xyz="0.0675 0.2575 -0.82" rpy="0 0 0"/>
+        <geometry>
+          <sphere radius="0.03"/>
+        </geometry>
+      </collision>
+      <collision>
+        <origin xyz="0.0675 -0.2575 -0.82" rpy="0 0 0"/>
+        <geometry>
+          <sphere radius="0.03"/>
+        </geometry>
+      </collision>
+      <collision>
+        <origin xyz="-0.4475 0.2575 -0.82" rpy="0 0 0"/>
+        <geometry>
+          <sphere radius="0.03"/>
+        </geometry>
+      </collision>
+      <collision>
+        <origin xyz="-0.4475 -0.2575 -0.82" rpy="0 0 0"/>
+        <geometry>
+          <sphere radius="0.03"/>
+        </geometry>
+      </collision>
+      <inertial>
+        <mass value="40" />
+        <origin xyz="-0.19 0 -0.435" rpy="0 0 0"/>
+        <xacro:nxa_box_inertia_def x="0.585" y="0.585" z="0.72" mass="40"/>
+      </inertial>
+    </link>
+    <joint name="base_to_waist" type="fixed">
+      <parent link="nextage_base"/>
+      <child link="WAIST"/>
+    </joint>
+  </xacro:macro>
 </robot>

File: nextagea_description/urdf/nextagea.urdf.xacro (robot description, xacro)
@@ -14,17 +14,31 @@
        xmlns:physics="http://playerstage.sourceforge.net/gazebo/xmlschema/#physics"
        xmlns:xacro="http://www.ros.org/wiki/xacro">
+  <!-- Include files for vanilla base -->
   <xacro:include filename="$(find nextagea_description)/urdf/general/materials.xacro" />
   <xacro:include filename="$(find nextagea_description)/urdf/general/common.xacro" />
-  <!-- Include the nextagea base, robot torso, and tools -->
   <xacro:include filename="$(find nextagea_description)/urdf/base/nextagea_base.xacro" />
   <xacro:include filename="$(find nextagea_description)/urdf/robot/nextagea_robot.xacro" />
   <xacro:include filename="$(find nextagea_description)/urdf/tool/nxao_gz_camera.xacro" />
-  <!-- Include extensions here -->
-  <!-- e.g. <xacro:include filename="$(find nextage_extensions)/urdf/intel_realsense.xacro" /> -->
+  <!-- Include files for extensions here -->
+  <xacro:include filename="$(find nextage_extensions)/urdf/intel_realsense.xacro" />
   <xacro:include filename="$(find nextage_extensions)/urdf/imu.xacro" />
-  <!-- <xacro:include filename="$(find nextage_extensions)/urdf/hexe.xacro" /> -->
-  <!-- <xacro:include filename="$(find nextage_extensions)/urdf/robotiq_140_gripper.xacro" />
-  <xacro:include filename="$(find nextage_extensions)/urdf/robotiq_85_gripper.xacro" /> -->
-  <!-- <xacro:include filename="$(find nextage_extensions)/urdf/robolimb.xacro" /> -->
+  <xacro:include filename="$(find nextage_extensions)/urdf/hexe.xacro" />
+  <xacro:include filename="$(find nextage_extensions)/urdf/robotiq_140_gripper.xacro" />
+  <xacro:include filename="$(find nextage_extensions)/urdf/robotiq_85_gripper.xacro" />
+  <xacro:include filename="$(find nextage_extensions)/urdf/robolimb.xacro" />
   <xacro:include filename="$(find nextage_extensions)/urdf/kinect.xacro" />
+  <!-- Include the nextagea base, robot torso, and tools -->
+  <xacro:nextagea_robot/>
+  <xacro:nextagea_base/>
+  <xacro:nextagea_tools use_hand_cameras="true" use_ft_sensors="true"/>
+  <!-- Include files for extensions here -->
+  <!-- Sensors -->
+  <xacro:intel_realsense/>
+  <xacro:imu/>
+  <xacro:nx_kinect/>
+  <!-- <xacro:hex_e/> -->
+  <!-- Actuators -->
+  <!-- <xacro:robotiq_140/>
+  <xacro:robotiq_85/>
+  <xacro:robolimb/> -->
 </robot>

File: nextagea_description/urdf/robot/nextagea_robot.xacro (robot description, xacro)
@@ -2,645 +2,646 @@
 <robot xmlns:xacro="http://ros.org/wiki/xacro">
   <xacro:include filename="$(find nextagea_description)/urdf/general/common.xacro" />
-  <xacro:property name="namespace" default="/nextagea/" />
-  <xacro:property name="nextagea_gazebo_ros_control" default="true" />
-  <xacro:gazebo_nx_link name="WAIST" color="Black" />
-  <link name="WAIST">
-    <visual>
-      <origin xyz="0 0 0" rpy="0 0 0"/>
-      <geometry>
-	      <mesh filename="package://nextagea_description/urdf/meshes/WAIST_Link_mesh.dae"/>
-      </geometry>
-    </visual>
-    <collision>
-      <origin xyz="0.0 0 0.098" rpy="0 0 0"/>
-      <geometry>
-        <cylinder length="0.376" radius="0.06"/>
-      </geometry>
-    </collision>
-    <inertial>
-      <mass value="5" />
-      <origin xyz="0 0 0.15" rpy="0 0 0"/>
-      <xacro:nxa_box_inertia_def x="0.2" y="0.2" z="0.3" mass="5"/>
-    </inertial>
-  </link>
-  <xacro:gazebo_nx_link name="CHEST_JOINT0_Link" color="Black" />
-  <link name="CHEST_JOINT0_Link">
-    <visual>
-      <origin xyz="0 0 0" rpy="0 0 0"/>
-      <geometry>
-	      <mesh filename="package://nextagea_description/urdf/meshes/CHEST_JOINT0_Link_mesh.dae"/>
-      </geometry>
-    </visual>
-    <collision>
-      <origin xyz="0 0 0.1575" rpy="0 0 0"/>
-      <geometry>
-        <cylinder length="0.385" radius="0.08"/>
-      </geometry>
-    </collision>
-    <collision>
-      <origin xyz="0.04 0.135 0.0423" rpy="0 0 0"/>
-      <geometry>
-        <cylinder length="0.09" radius="0.05"/>
-      </geometry>
-    </collision>
-    <collision>
-      <origin xyz="0.04 -0.135 0.0423" rpy="0 0 0"/>
-      <geometry>
-        <cylinder length="0.09" radius="0.05"/>
-      </geometry>
-    </collision>
-    <collision>
-      <origin xyz="0 0 0.055" rpy="0 0 0"/>
-      <geometry>
-        <box size="0.23 0.18 0.12"/>
-      </geometry>
-    </collision>
-    <collision>
-      <origin xyz="-0.04 0 0.2325" rpy="0 0 0"/>
-      <geometry>
-        <box size="0.25 0.18 0.245"/>
-      </geometry>
-    </collision>
-    <collision>
-      <origin xyz="-0.1525 0 0.279" rpy="0 0 0"/>
-      <geometry>
-        <box size="0.17 0.29 0.225"/>
-      </geometry>
-    </collision>
-    <collision>
-      <origin xyz="0.03 0 0.315" rpy="0 0 0"/>
-      <geometry>
-        <box size="0.085 0.5 0.0365"/>
-      </geometry>
-    </collision>
-    <inertial>
-      <mass value="10.0" />
-      <origin xyz="0 0 0.2" rpy="0 -0 0"/>
-      <xacro:nxa_box_inertia_def x="0.25" y="0.25" z="0.3" mass="10"/>
-    </inertial>
-  </link>
-  <xacro:gazebo_nx_link name="HEAD_JOINT0_Link" color="Black" />
-  <link name="HEAD_JOINT0_Link">
-    <visual>
-      <origin xyz="0 0 0" rpy="0 0 0"/>
-      <geometry>
-	      <mesh filename="package://nextagea_description/urdf/meshes/HEAD_JOINT0_Link_mesh.dae"/>
-      </geometry>
-    </visual>
-    <collision>
-      <origin xyz="0 0.01 0.08" rpy="1.57079 0 0"/>
-      <geometry>
-        <cylinder length="0.135" radius="0.035"/>
-      </geometry>
-    </collision>
-     <inertial>
-      <mass value="0.317929" />
-      <origin xyz="0 0.00547848 0" rpy="0 -0 0"/>
-      <xacro:nxa_box_inertia_def x="0.1" y="0.1" z="0.1" mass="0.317929"/>
-    </inertial>
-  </link>
-  <xacro:gazebo_nx_link name="HEAD_JOINT1_Link" color="Black" />
-  <link name="HEAD_JOINT1_Link">
-    <visual>
-      <origin xyz="0 0 0" rpy="0 0 0"/>
-      <geometry>
-	      <mesh filename="package://nextagea_description/urdf/meshes/HEAD_JOINT1_Link_mesh.dae"/>
-      </geometry>
-    </visual>
-    <collision>
-      <origin xyz="-0.05 0 0.12" rpy="0 0.26 0"/>
-      <geometry>
-        <box size="0.27 0.22 0.115"/>
-      </geometry>
-    </collision>
-    <inertial>
-      <mass value="0.4" />
-      <origin xyz="-0.05 0 0.12" rpy="0 0.26 0"/>
-      <xacro:nxa_box_inertia_def x="0.27" y="0.22" z="0.115" mass="0.4"/>
-    </inertial>
-  </link>
-  <xacro:gazebo_nx_link name="LARM_JOINT0_Link" color="Black" />
-  <link name="LARM_JOINT0_Link">
-    <visual>
-      <origin xyz="0 0 0" rpy="0 0 0"/>
-      <geometry>
-	      <mesh filename="package://nextagea_description/urdf/meshes/LARM_JOINT0_Link_mesh.dae"/>
-      </geometry>
-    </visual>
-    <collision>
-      <origin xyz="0 0.00775 0.095" rpy="0 0 0"/>
-      <geometry>
-        <box size="0.1 0.0815 0.19"/>
-      </geometry>
-    </collision>
-    <collision>
-      <origin xyz="0 0.0875 0.066" rpy="1.57079 0 0"/>
-      <geometry>
-        <cylinder length="0.175" radius="0.042"/>
-      </geometry>
-    </collision>
-    <collision>
-      <origin xyz="0 0.125 0.145" rpy="-0.7 0 0"/>
-      <geometry>
-        <box size="0.048 0.1 0.035"/>
-      </geometry>
-    </collision>
-    <inertial>
-      <mass value="1.32626" />
-      <origin xyz="0.0 0.05 0.05" rpy="0 -0 0"/>
-      <inertia ixx="0.00207537" ixy="0.00011276" ixz="8.927e-05" iyy="0.00240295" iyz="-4.57e-05" izz="0.00141912"/>
-    </inertial>
-  </link>
-  <xacro:gazebo_nx_link name="LARM_JOINT1_Link" color="Black" />
-  <link name="LARM_JOINT1_Link">
-    <visual>
-      <origin xyz="0 0 0" rpy="0 0 0"/>
-      <geometry>
-	      <mesh filename="package://nextagea_description/urdf/meshes/LARM_JOINT1_Link_mesh.dae"/>
-      </geometry>
-    </visual>
-    <collision>
-      <origin xyz="-0.043 0.12 -0.13" rpy="0 0.3 0"/>
-      <geometry>
-        <box size="0.08 0.11 0.28"/>
-      </geometry>
-    </collision>
-    <collision>
-      <origin xyz="-0.03 0.0518 -0.236" rpy="0 0.45 0"/>
-      <geometry>
-        <box size="0.122 0.0338 0.062"/>
-      </geometry>
-    </collision>
-     <inertial>
-      <mass value="1.14898" />
-      <origin xyz="-0.04 0.1 -0.12" rpy="0 -0 0"/>
-      <inertia ixx="0.0154168" ixy="9.95417e-07" ixz="3.38147e-06" iyy="0.0147117" iyz="0.00213719" izz="0.0012658"/>
-    </inertial>
-  </link>
-  <xacro:gazebo_nx_link name="LARM_JOINT2_Link" color="Black" />
-  <link name="LARM_JOINT2_Link">
-    <visual>
-      <origin xyz="0 0 0" rpy="0 0 0"/>
-      <geometry>
-	      <mesh filename="package://nextagea_description/urdf/meshes/LARM_JOINT2_Link_mesh.dae"/>
-      </geometry>
-    </visual>
-    <collision>
-      <origin xyz="0 0.025 0" rpy="1.57079 0 0"/>
-      <geometry>
-        <cylinder length="0.11" radius="0.049"/>
-      </geometry>
-    </collision>
-    <collision>
-      <origin xyz="0.0945 0.015 -0.03" rpy="0 0 0"/>
-      <geometry>
-        <box size="0.119 0.125 0.1"/>
-      </geometry>
-    </collision>
-    <collision>
-      <origin xyz="0.17 0 -0.03" rpy="0 1.57079 0"/>
-      <geometry>
-        <cylinder length="0.04" radius="0.047"/>
-      </geometry>
-    </collision>
-    <inertial>
-      <mass value="0.577518" />
-      <origin xyz="0.1 0.01167107 -0.04" rpy="0 -0 0"/>
-      <inertia ixx="0.00143966" ixy="-3e-07" ixz="1.2e-06" iyy="0.00141763" iyz="-7.596e-05" izz="0.0001972"/>
-    </inertial>
-  </link>
-  <xacro:gazebo_nx_link name="LARM_JOINT3_Link" color="Black" />
-  <link name="LARM_JOINT3_Link">
-    <visual>
-      <origin xyz="0 0 0" rpy="0 0 0"/>
-      <geometry>
-	      <mesh filename="package://nextagea_description/urdf/meshes/LARM_JOINT3_Link_mesh.dae"/>
-      </geometry>
-    </visual>
-    <collision>
-      <origin xyz="0.1495 -0.003 0" rpy="1.57079 0 0"/>
-      <geometry>
-        <cylinder length="0.12" radius="0.035"/>
-      </geometry>
-    </collision>
-    <collision>
-      <origin xyz="0.075 0.0 0.018" rpy="0 1.57079 0"/>
-      <geometry>
-        <cylinder length="0.15" radius="0.04"/>
-      </geometry>
-    </collision>
-    <collision>
-      <origin xyz="0.0585 0.01 0.0185" rpy="0 0 0"/>
-      <geometry>
-        <box size="0.093 0.112 0.037"/>
-      </geometry>
-    </collision>
-    <inertial>
-      <mass value="0.457418" />
-      <origin xyz="0.1 -0.00395812 -0.00273" rpy="0 -0 0"/>
-      <inertia ixx="0.00069205" ixy="3e-08" ixz="5.2e-07" iyy="0.00068903" iyz="-1.915e-05" izz="0.00013509"/>
-    </inertial>
-  </link>
-  <xacro:gazebo_nx_link name="LARM_JOINT4_Link" color="Black" />
-  <link name="LARM_JOINT4_Link">
-    <visual>
-      <origin xyz="0 0 0" rpy="0 0 0"/>
-      <geometry>
-	      <mesh filename="package://nextagea_description/urdf/meshes/LARM_JOINT4_Link_mesh.dae"/>
-      </geometry>
-    </visual>
-    <collision>
-      <origin xyz="0 -0.002 -0.06" rpy="0 0 0"/>
-      <geometry>
-        <box size="0.04 0.118 0.06"/>
-      </geometry>
-    </collision>
-    <collision>
-      <origin xyz="0 0 -0.08" rpy="0 0 0"/>
-      <geometry>
-        <cylinder length="0.08" radius="0.037"/>
-      </geometry>
-    </collision>
-    <inertial>
-      <mass value="0.418434" />
-      <origin xyz="0.00243131 0.00379733 -0.0577036" rpy="0 -0 0"/>
-      <inertia ixx="0.00052016" ixy="1.69e-06" ixz="7.9e-06" iyy="0.00050569" iyz="-5.377e-05" izz="0.00014004"/>
-    </inertial>
-  </link>
-  <xacro:gazebo_nx_link name="LARM_JOINT5_Link" color="Black" />
-  <link name="LARM_JOINT5_Link">
-    <visual>
-      <origin xyz="0 0 0" rpy="0 0 0"/>
-      <geometry>
-	      <mesh filename="package://nextagea_description/urdf/meshes/LARM_JOINT5_Link_mesh.dae"/>
-      </geometry>
-    </visual>
-    <collision>
-      <origin xyz="0 0 0.0065" rpy="0 0 0"/>
-      <geometry>
-        <cylinder length="0.013" radius="0.037"/>
-      </geometry>
-    </collision>
-    <inertial>
-      <mass value="1.05156" />
-      <origin xyz="0.0 0.0 -0.08" rpy="0 -0 0"/>
-      <inertia ixx="0.00194072" ixy="1.1e-07" ixz="-0.00042482" iyy="0.00209392" iyz="1.2e-07" izz="0.00035788"/>
-    </inertial>
-  </link>
-  <xacro:gazebo_nx_link name="RARM_JOINT0_Link" color="Black" />
-  <link name="RARM_JOINT0_Link">
-    <visual>
-      <origin xyz="0 0 0" rpy="0 0 0"/>
-      <geometry>
-	      <mesh filename="package://nextagea_description/urdf/meshes/RARM_JOINT0_Link_mesh.dae"/>
-      </geometry>
-    </visual>
-    <collision>
-      <origin xyz="0 -0.00775 0.095" rpy="0 0 0"/>
-      <geometry>
-        <box size="0.1 0.0815 0.19"/>
-      </geometry>
-    </collision>
-    <collision>
-      <origin xyz="0 -0.0875 0.066" rpy="1.57079 0 0"/>
-      <geometry>
-        <cylinder length="0.175" radius="0.042"/>
-      </geometry>
-    </collision>
-    <collision>
-      <origin xyz="0 -0.125 0.145" rpy="0.7 0 0"/>
-      <geometry>
-        <box size="0.048 0.1 0.035"/>
-      </geometry>
-    </collision>
-    <inertial>
-      <mass value="1.32626" />
-      <origin xyz="0.0 -0.05 0.05" rpy="0 -0 0"/>
-      <inertia ixx="0.00207537" ixy="-0.00011276" ixz="8.927e-05" iyy="0.00240295" iyz="4.57e-05" izz="0.00141912"/>
-    </inertial>
-  </link>
-  <xacro:gazebo_nx_link name="RARM_JOINT1_Link" color="Black" />
-  <link name="RARM_JOINT1_Link">
-    <visual>
-      <origin xyz="0 0 0" rpy="0 0 0"/>
-      <geometry>
-	      <mesh filename="package://nextagea_description/urdf/meshes/RARM_JOINT1_Link_mesh.dae"/>
-      </geometry>
-    </visual>
-    <collision>
-      <origin xyz="-0.043 -0.12 -0.13" rpy="0 0.3 0"/>
-      <geometry>
-        <box size="0.08 0.11 0.28"/>
-      </geometry>
-    </collision>
-    <collision>
-      <origin xyz="-0.03 -0.0518 -0.236" rpy="0 0.45 0"/>
-      <geometry>
-        <box size="0.122 0.0338 0.062"/>
-      </geometry>
-    </collision>
-    <inertial>
-      <mass value="1.14898" />
-      <origin xyz="-0.04 -0.1 -0.12" rpy="0 -0 0"/>
-      <inertia ixx="0.0154168" ixy="-9.95417e-07" ixz="3.38147e-06" iyy="0.0147117" iyz="-0.00213719" izz="0.0012658"/>
-    </inertial>
-  </link>
-  <xacro:gazebo_nx_link name="RARM_JOINT2_Link" color="Black" />
-  <link name="RARM_JOINT2_Link">
-    <visual>
-      <origin xyz="0 0 0" rpy="0 0 0"/>
-      <geometry>
-	      <mesh filename="package://nextagea_description/urdf/meshes/RARM_JOINT2_Link_mesh.dae"/>
-      </geometry>
-    </visual>
-    <collision>
-      <origin xyz="0 -0.025 0" rpy="1.57079 0 0"/>
-      <geometry>
-        <cylinder length="0.11" radius="0.049"/>
-      </geometry>
-    </collision>
-    <collision>
-      <origin xyz="0.0945 -0.015 -0.03" rpy="0 0 0"/>
-      <geometry>
-        <box size="0.119 0.125 0.1"/>
-      </geometry>
-    </collision>
-    <collision>
-      <origin xyz="0.17 0 -0.03" rpy="0 1.57079 0"/>
-      <geometry>
-        <cylinder length="0.04" radius="0.047"/>
-      </geometry>
-    </collision>
-    <inertial>
-      <mass value="0.577518" />
-      <origin xyz="0.1 -0.01167107 -0.04" rpy="0 -0 0"/>
-      <inertia ixx="0.00143966" ixy="3e-07" ixz="1.2e-06" iyy="0.00141763" iyz="7.596e-05" izz="0.0001972"/>
-    </inertial>
-  </link>
-  <xacro:gazebo_nx_link name="RARM_JOINT3_Link" color="Black" />
-  <link name="RARM_JOINT3_Link">
-    <visual>
-      <origin xyz="0 0 0" rpy="0 0 0"/>
-      <geometry>
-	      <mesh filename="package://nextagea_description/urdf/meshes/RARM_JOINT3_Link_mesh.dae"/>
-      </geometry>
-    </visual>
-    <collision>
-      <origin xyz="0.1495 -0.003 0" rpy="1.57079 0 0"/>
-      <geometry>
-        <cylinder length="0.12" radius="0.035"/>
-      </geometry>
-    </collision>
-    <collision>
-      <origin xyz="0.075 0.0 0.018" rpy="0 1.57079 0"/>
-      <geometry>
-        <cylinder length="0.15" radius="0.04"/>
-      </geometry>
-    </collision>
-    <collision>
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