Commit message: added macros to wrap around each object

File: nextagea_description/urdf/tool/nxao_gz_camera.xacro (robot description, xacro)
@@ -5,298 +5,295 @@
 		Values in Gazebo plugin are originally copied from http://gazebosim.org/tutorials?tut=ros_gzplugins#camera
 		and only partially tailored as of May 2017 -->
-	<!-- Properties -->
-	<xacro:property name="M_PI" value="3.1415926535897931" />
-	<xacro:property name="jnt_head_camera_displacement_x" value="0.0175" />
-	<xacro:property name="jnt_head_camera_displacement_y" value="0.0725" />
-	<xacro:property name="jnt_head_camera_displacement_z" value="0.105" />
-	<xacro:property name="jnt_head_camera_rot_y" value="0.25" />
-	<xacro:property name="link_head_camera_rot_z" value="0.05" />
-	<xacro:property name="jnt_hand_camera_displacement_x" value="0.0525" />
-	<xacro:property name="jnt_hand_camera_displacement_y" value="0.0525" />
-	<xacro:property name="jnt_hand_camera_displacement_z" value="0.0" />
-	<xacro:property name="jnt_hand_camera_rot_y" value="1.5708" />
-	<xacro:property name="link_hand_camera_rot_z" value="0.0" />
-	<xacro:property name="arm_tip" value="ARM_JOINT5_Link" />
-	<!-- Arguments  -->
-	<xacro:arg name="fixed_base" default="true" />
-	<xacro:arg name="use_hand_cameras" default="true"/>
-	<xacro:arg name="use_ft_sensors" default="true"/>
-	<xacro:arg name="use_cables_right" default="true"/>
-	<xacro:arg name="use_cables_left" default="true"/>
-	<!-- Camera macro -->
-	<xacro:macro name="nxao_camera" params="prefix parent">
-    <xacro:if value="${prefix == 'L'}">
-      <xacro:property name="m" value="+1" />
-    </xacro:if>
-    <xacro:if value="${prefix == 'R'}">
-      <xacro:property name="m" value="-1" />
-    </xacro:if>
-    <xacro:gazebo_nx_link name="${prefix}ARM_camera_Link" color="Black" />
-    <link name="${prefix}ARM_camera_Link">
-      <visual>
+  <xacro:macro name="nextagea_tools" params="fixed_base:= true use_hand_cameras:=false
+                      use_ft_sensors:=false use_cables_right:=true use_cables_left:=true">
+    <!-- Properties -->
+    <xacro:property name="M_PI" value="3.1415926535897931" />
+    <xacro:property name="jnt_head_camera_displacement_x" value="0.0175" />
+    <xacro:property name="jnt_head_camera_displacement_y" value="0.0725" />
+    <xacro:property name="jnt_head_camera_displacement_z" value="0.105" />
+    <xacro:property name="jnt_head_camera_rot_y" value="0.25" />
+    <xacro:property name="link_head_camera_rot_z" value="0.05" />
+    <xacro:property name="jnt_hand_camera_displacement_x" value="0.0525" />
+    <xacro:property name="jnt_hand_camera_displacement_y" value="0.0525" />
+    <xacro:property name="jnt_hand_camera_displacement_z" value="0.0" />
+    <xacro:property name="jnt_hand_camera_rot_y" value="1.5708" />
+    <xacro:property name="link_hand_camera_rot_z" value="0.0" />
+    <xacro:property name="arm_tip" value="ARM_JOINT5_Link" />
+    <!-- Camera macro -->
+    <xacro:macro name="nxao_camera" params="prefix parent">
+      <xacro:if value="${prefix == 'L'}">
+        <xacro:property name="m" value="+1" />
+      </xacro:if>
+      <xacro:if value="${prefix == 'R'}">
+        <xacro:property name="m" value="-1" />
+      </xacro:if>
+      <xacro:gazebo_nx_link name="${prefix}ARM_camera_Link" color="Black" />
+      <link name="${prefix}ARM_camera_Link">
+        <visual>
+          <origin xyz="0 0 0" rpy="0 0 0"/>
+          <geometry>
+            <mesh filename="package://nextagea_description/urdf/meshes/${prefix}_CAM.dae"/>
+          </geometry>
+        </visual>
+        <collision>
+          <origin xyz="0 0 -0.025" rpy="0 0 0"/>
+          <geometry>
+            <cylinder length="0.05" radius="0.037"/>
+          </geometry>
+        </collision>
+        <collision>
+          <origin xyz="0.0525 ${m * 0.029} -0.02" rpy="0 0 0"/>
+          <geometry>
+            <box size="0.057 0.106 0.042"/>
+          </geometry>
+        </collision>
+        <inertial>
+          <mass value="1.05156" />
+          <origin xyz="0.0 0.0 -0.08" rpy="0 -0 0"/>
+          <inertia ixx="0.00194072" ixy="${m * 1.1e-07}" ixz="-0.00042482" iyy="0.00209392" iyz="${m * 1.2e-07}" izz="0.00035788"/>
+        </inertial>
+      </link>
+      <joint name="${prefix}ARM_JOINT6" type="fixed">
+        <parent link="${parent}"/>
+        <child link="${prefix}ARM_camera_Link"/>
         <origin xyz="0 0 0" rpy="0 0 0"/>
-        <geometry>
-          <mesh filename="package://nextagea_description/urdf/meshes/${prefix}_CAM.dae"/>
-        </geometry>
-      </visual>
-      <collision>
-        <origin xyz="0 0 -0.025" rpy="0 0 0"/>
-        <geometry>
-          <cylinder length="0.05" radius="0.037"/>
-        </geometry>
-      </collision>
-      <collision>
-        <origin xyz="0.0525 ${m * 0.029} -0.02" rpy="0 0 0"/>
-        <geometry>
-          <box size="0.057 0.106 0.042"/>
-        </geometry>
-      </collision>
-      <inertial>
-        <mass value="1.05156" />
-        <origin xyz="0.0 0.0 -0.08" rpy="0 -0 0"/>
-        <inertia ixx="0.00194072" ixy="${m * 1.1e-07}" ixz="-0.00042482" iyy="0.00209392" iyz="${m * 1.2e-07}" izz="0.00035788"/>
-      </inertial>
-    </link>
-    <joint name="${prefix}ARM_JOINT6" type="fixed">
-      <parent link="${parent}"/>
-      <child link="${prefix}ARM_camera_Link"/>
-      <origin xyz="0 0 0" rpy="0 0 0"/>
-      <axis xyz="0 0 1"/>
-    </joint>
+        <axis xyz="0 0 1"/>
+      </joint>
+      <xacro:camera_joint_link_gzplugin
+        camera_name="CAMERA_HAND_${prefix}" link_parent="${parent}"
+        jnt_displacement_x="${jnt_hand_camera_displacement_x}"
+        jnt_displacement_y="${m * jnt_hand_camera_displacement_y}"
+        jnt_displacement_z="${jnt_hand_camera_displacement_z}"
+        jnt_rotation_x="0" jnt_rotation_y="${jnt_hand_camera_rot_y}" jnt_rotation_z="0"
+        link_displacement_x="0.0325" link_displacement_y="0" link_displacement_z="0"
+        link_rotation_x="0" link_rotation_y="${M_PI/2}" link_rotation_z="-${link_hand_camera_rot_z}" />
+    </xacro:macro>
+    <!-- FT Sensor macro -->
+    <xacro:macro name="nxao_ft_sensor" params="prefix parent">
+      <xacro:if value="${prefix == 'L'}">
+        <xacro:property name="m" value="+1" />
+        <xacro:property name="ft_side" value="left" />
+      </xacro:if>
+      <xacro:if value="${prefix == 'R'}">
+        <xacro:property name="m" value="-1" />
+        <xacro:property name="ft_side" value="right" />
+      </xacro:if>
+      <xacro:gazebo_nx_link name="${prefix}ARM_ft_Link" color="LightGrey" />
+      <link name="${prefix}ARM_ft_Link_base">
+        <visual>
+          <origin xyz="0 0 0.0185" rpy="0 0 0"/>
+          <geometry>
+            <cylinder length="0.037" radius="0.035"/>
+          </geometry>
+          <material name="LightGrey">
+            <color rgba="0.6 0.6 0.6 1.0"/>
+          </material>
+        </visual>
+        <collision>
+          <origin xyz="0 0 0.0185" rpy="0 0 0"/>
+          <geometry>
+            <cylinder length="0.037" radius="0.04"/>
+          </geometry>
+        </collision>
+        <!-- TODO: The inertial values are copied from ARM_JOINT5_Link. Replace with proper values. -->
+        <inertial>
+          <mass value="1.05156" />
+          <origin xyz="0.0 0.0 -0.08" rpy="0 -0 0"/>
+          <inertia ixx="0.00194072" ixy="1.1e-07" ixz="-0.00042482" iyy="0.00209392" iyz="1.2e-07" izz="0.00035788"/>
+        </inertial>
+      </link>
+      <joint name="${prefix}ARM_ft_joint" type="fixed">
+        <parent link="${parent}"/>
+        <child link="${prefix}ARM_ft_Link_base"/>
+        <origin xyz="0 0 -0.037" rpy="0 0 0"/>
+        <axis xyz="0 0 1"/>
+      </joint>
+      <link name="${prefix}ARM_ft_Sensor_Link">
+        <inertial>
+          <mass value="0.0001" />
+          <origin xyz="0 0 0" rpy="0 0 0"/>
+          <xacro:nxa_sphere_inertia_def radius="0.0001" mass="0.0001"/>
+        </inertial>
+      </link>
+      <link name="${prefix}ARM_ft_Link">
+        <inertial>
+          <mass value="0.0001" />
+          <origin xyz="0 0 0" rpy="0 0 0"/>
+          <xacro:nxa_sphere_inertia_def radius="0.0001" mass="0.0001"/>
+        </inertial>
+      </link>
+      <joint name="${prefix}ARM_ft_sensor_joint" type="fixed">
+        <parent link="${prefix}ARM_ft_Link_base"/>
+        <child link="${prefix}ARM_ft_Sensor_Link"/>
+        <origin xyz="0 0 0" rpy="0 3.1415 1.57"/>
+        <axis xyz="0 0 1"/>
+      </joint>
+      <joint name="${prefix}ARM_ft_sensor_offset_joint" type="fixed">
+        <parent link="${prefix}ARM_ft_Sensor_Link"/>
+        <child link="${prefix}ARM_ft_Link"/>
+        <origin xyz="0 0 0" rpy="0 3.1415 1.57"/>
+        <axis xyz="0 0 1"/>
+      </joint>
+      <gazebo reference="${prefix}ARM_ft_sensor_joint">
+        <disableFixedJointLumping>true</disableFixedJointLumping>
+        <sensor name="${prefix}ARM_ft_sensor" type="force_torque">
+          <force_torque>
+            <frame>parent</frame>
+            <measure_direction>child_to_parent</measure_direction>
+          </force_torque>
+        </sensor>
+      </gazebo>
+      <gazebo>
+          <plugin name="${prefix}ARM_ft_sensor" filename="libgazebo_ros_ft_sensor.so">
+              <updateRate>500.0</updateRate>
+              <topicName>ft_${ft_side}/data</topicName>
+              <jointName>${prefix}ARM_ft_sensor_joint</jointName>
+          </plugin>
+      </gazebo>
+    </xacro:macro>
+    <!-- Adding camera for simulation -->
+    <xacro:macro name="camera_joint_link_gzplugin"
+      params="camera_name link_parent jnt_displacement_x jnt_displacement_y jnt_displacement_z jnt_rotation_x jnt_rotation_y jnt_rotation_z link_displacement_x link_displacement_y link_displacement_z link_rotation_x link_rotation_y link_rotation_z">
+      <joint name="${camera_name}" type="fixed">
+        <origin
+          xyz="${jnt_displacement_x} ${jnt_displacement_y} ${jnt_displacement_z}"
+          rpy="${jnt_rotation_x} ${jnt_rotation_y} ${jnt_rotation_z}" />
+        <parent link="${link_parent}" />
+        <child link="${camera_name}_Link" />
+      </joint>
+      <link name="${camera_name}_Link">
+        <visual>
+          <origin
+            xyz="${link_displacement_x} ${link_displacement_y} ${link_displacement_z}"
+            rpy="${link_rotation_x} ${link_rotation_y} ${link_rotation_z}" />
+          <geometry>
+            <cylinder length="0.01" radius="0.015" />
+          </geometry>
+          <material name="Blue" />
+        </visual>
+        <inertial>
+          <origin xyz="0 0 0" rpy="0 0 0" />
+          <mass value="1e-6" />
+          <inertia ixx="1e-12" ixy="0.0" ixz="0.0" iyy="1e-12" iyz="0.0"
+            izz="1e-12" />
+        </inertial>
+      </link>
+      <gazebo reference="${camera_name}_Link">
+        <sensor type="camera" name="${camera_name}">
+          <update_rate>30.0</update_rate>
+          <camera name="${camera_name}">
+            <horizontal_fov>1.3962634</horizontal_fov>
+            <image>
+              <width>800</width>
+              <height>800</height>
+              <format>R8G8B8</format>
+            </image>
+            <clip>
+              <near>0.1</near>
+              <far>30</far>
+            </clip>
+            <noise>
+              <type>gaussian</type>
+              <!-- Noise is sampled independently per pixel on each frame. That pixel's
+                noise value is added to each of its color channels, which at that point lie
+                in the range [0,1]. -->
+              <mean>0.0</mean>
+              <stddev>0.007</stddev>
+            </noise>
+          </camera>
+          <plugin name="camera_controller" filename="libgazebo_ros_camera.so">
+            <alwaysOn>true</alwaysOn>
+            <updateRate>0.0</updateRate>
+            <cameraName>${camera_name}</cameraName>
+            <imageTopicName>image_raw</imageTopicName>
+            <cameraInfoTopicName>camera_info</cameraInfoTopicName>
+            <frameName>${camera_name}_Link_frame</frameName>
+            <hackBaseline>0.07</hackBaseline>
+            <distortionK1>0.0</distortionK1>
+            <distortionK2>0.0</distortionK2>
+            <distortionK3>0.0</distortionK3>
+            <distortionT1>0.0</distortionT1>
+            <distortionT2>0.0</distortionT2>
+          </plugin>
+        </sensor>
+      </gazebo>
+    </xacro:macro>
+    <!-- NOTE: The poses of headmount and hand cameras are NOT precisely adjusted to
+          the 3D model nor the actual hardware config. These configs
+          are meant for a rapid prototyping only.
+    -->
     <xacro:camera_joint_link_gzplugin
-      camera_name="CAMERA_HAND_${prefix}" link_parent="${parent}"
-      jnt_displacement_x="${jnt_hand_camera_displacement_x}"
-      jnt_displacement_y="${m * jnt_hand_camera_displacement_y}"
-      jnt_displacement_z="${jnt_hand_camera_displacement_z}"
-      jnt_rotation_x="0" jnt_rotation_y="${jnt_hand_camera_rot_y}" jnt_rotation_z="0"
-      link_displacement_x="0.0325" link_displacement_y="0" link_displacement_z="0"
-      link_rotation_x="0" link_rotation_y="${M_PI/2}" link_rotation_z="-${link_hand_camera_rot_z}" />
+        camera_name="CAMERA_HEAD_L" link_parent="HEAD_JOINT1_Link"
+        jnt_displacement_x="${jnt_head_camera_displacement_x}" jnt_displacement_y="${jnt_head_camera_displacement_y}" jnt_displacement_z="${jnt_head_camera_displacement_z}"
+        jnt_rotation_x="0" jnt_rotation_y="${jnt_head_camera_rot_y}" jnt_rotation_z="0"
+        link_displacement_x="0.0325" link_displacement_y="0" link_displacement_z="0"
+        link_rotation_x="0" link_rotation_y="${M_PI/2}" link_rotation_z="-${link_head_camera_rot_z}" />
+    <xacro:camera_joint_link_gzplugin
+        camera_name="CAMERA_HEAD_R" link_parent="HEAD_JOINT1_Link"
+        jnt_displacement_x="${jnt_head_camera_displacement_x}" jnt_displacement_y="-${jnt_head_camera_displacement_y}" jnt_displacement_z="${jnt_head_camera_displacement_z}"
+        jnt_rotation_x="0" jnt_rotation_y="${jnt_head_camera_rot_y}" jnt_rotation_z="0"
+        link_displacement_x="0.0325" link_displacement_y="0" link_displacement_z="0"
+        link_rotation_x="0" link_rotation_y="${M_PI/2}" link_rotation_z="${link_head_camera_rot_z}" />
+    <!-- Deal with arguments -->
+    <xacro:if value="${fixed_base}">
+      <link name="world"/>
+      <joint name="fixed" type="fixed">
+        <parent link="world"/>
+        <child link="base_link"/>
+        <origin xyz="0 0 0.85" rpy="0 0 0"/>
+      </joint>
+    </xacro:if>
+    <xacro:if value="${use_ft_sensors}">
+      <xacro:nxao_ft_sensor prefix="L" parent="L${arm_tip}" />
+      <xacro:nxao_ft_sensor prefix="R" parent="R${arm_tip}" />
+      <xacro:property name="arm_tip" value="ARM_ft_Link" />
+    </xacro:if>
+    <xacro:if value="${use_hand_cameras}">
+      <xacro:nxao_camera prefix="L" parent="L${arm_tip}" />
+      <xacro:nxao_camera prefix="R" parent="R${arm_tip}" />
+      <xacro:property name="arm_tip" value="ARM_camera_Link" />
+    </xacro:if>
+    <xacro:if value="${use_cables_left}">
+      <joint name="LARM_JOINT4_Link_cables_joint" type="fixed">
+        <parent link="LARM_JOINT4_Link"/>
+        <child link="LARM_JOINT4_Link_cables"/>
+        <origin xyz="0 0 0" rpy="0 0 0"/>
+        <axis xyz="0 0 1"/>
+      </joint>
+      <link name="LARM_JOINT4_Link_cables">
+        <inertial>
+          <mass value="0.01" />
+          <origin xyz="0 0 0" rpy="0 0 0"/>
+          <xacro:nxa_box_inertia_def x="0.016" y="0.006" z="0.012" mass="0.01"/>
+        </inertial>
+        <collision>
+          <origin xyz="0 0.08 -0.1" rpy="0 0 0"/>
+          <geometry>
+            <sphere radius="0.1"/>
+          </geometry>
+        </collision>
+      </link>
+    </xacro:if>
+    <xacro:if value="${use_cables_right}">
+      <joint name="RARM_JOINT4_Link_cables_joint" type="fixed">
+        <parent link="RARM_JOINT4_Link"/>
+        <child link="RARM_JOINT4_Link_cables"/>
+        <origin xyz="0 0 0" rpy="0 0 0"/>
+        <axis xyz="0 0 1"/>
+      </joint>
+      <link name="RARM_JOINT4_Link_cables">
+        <inertial>
+          <mass value="0.01" />
+          <origin xyz="0 0 0" rpy="0 0 0"/>
+          <xacro:nxa_box_inertia_def x="0.016" y="0.006" z="0.012" mass="0.01"/>
+        </inertial>
+        <collision>
+          <origin xyz="0 -0.08 -0.1" rpy="0 0 0"/>
+          <geometry>
+            <sphere radius="0.1"/>
+          </geometry>
+        </collision>
+      </link>
+    </xacro:if>
   </xacro:macro>
-  <!-- FT Sensor macro -->
-  <xacro:macro name="nxao_ft_sensor" params="prefix parent">
-    <xacro:if value="${prefix == 'L'}">
-      <xacro:property name="m" value="+1" />
-      <xacro:property name="ft_side" value="left" />
-    </xacro:if>
-    <xacro:if value="${prefix == 'R'}">
-      <xacro:property name="m" value="-1" />
-      <xacro:property name="ft_side" value="right" />
-    </xacro:if>
-    <xacro:gazebo_nx_link name="${prefix}ARM_ft_Link" color="LightGrey" />
-    <link name="${prefix}ARM_ft_Link_base">
-      <visual>
-        <origin xyz="0 0 0.0185" rpy="0 0 0"/>
-        <geometry>
-          <cylinder length="0.037" radius="0.035"/>
-        </geometry>
-        <material name="LightGrey">
-          <color rgba="0.6 0.6 0.6 1.0"/>
-        </material>
-      </visual>
-      <collision>
-        <origin xyz="0 0 0.0185" rpy="0 0 0"/>
-        <geometry>
-          <cylinder length="0.037" radius="0.04"/>
-        </geometry>
-      </collision>
-      <!-- TODO: The inertial values are copied from ARM_JOINT5_Link. Replace with proper values. -->
-      <inertial>
-        <mass value="1.05156" />
-        <origin xyz="0.0 0.0 -0.08" rpy="0 -0 0"/>
-        <inertia ixx="0.00194072" ixy="1.1e-07" ixz="-0.00042482" iyy="0.00209392" iyz="1.2e-07" izz="0.00035788"/>
-      </inertial>
-    </link>
-    <joint name="${prefix}ARM_ft_joint" type="fixed">
-      <parent link="${parent}"/>
-      <child link="${prefix}ARM_ft_Link_base"/>
-      <origin xyz="0 0 -0.037" rpy="0 0 0"/>
-      <axis xyz="0 0 1"/>
-    </joint>
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