Commit message: covid contact so committing but broken

File: nextagea_description/urdf/general/common.xacro (robot description, xacro)
@@ -39,4 +39,83 @@
             </gazebo>
         </xacro:macro>
+        <!-- Camera gazebo plugin -->
+        <!-- Properties -->
+        <xacro:property name="M_PI" value="3.1415926535897931" />
+        <xacro:property name="jnt_head_camera_displacement_x" value="0.0175" />
+        <xacro:property name="jnt_head_camera_displacement_y" value="0.0725" />
+        <xacro:property name="jnt_head_camera_displacement_z" value="0.105" />
+        <xacro:property name="jnt_head_camera_rot_y" value="0.25" />
+        <xacro:property name="link_head_camera_rot_z" value="0.05" />
+        <xacro:property name="jnt_hand_camera_displacement_x" value="0.0525" />
+        <xacro:property name="jnt_hand_camera_displacement_y" value="0.0525" />
+        <xacro:property name="jnt_hand_camera_displacement_z" value="0.0" />
+        <xacro:property name="jnt_hand_camera_rot_y" value="1.5708" />
+        <xacro:property name="link_hand_camera_rot_z" value="0.0" />
+        <xacro:macro name="camera_joint_link_gzplugin"
+        params="camera_name link_parent jnt_displacement_x jnt_displacement_y jnt_displacement_z jnt_rotation_x jnt_rotation_y jnt_rotation_z link_displacement_x link_displacement_y link_displacement_z link_rotation_x link_rotation_y link_rotation_z">
+            <joint name="${camera_name}" type="fixed">
+            <origin
+                xyz="${jnt_displacement_x} ${jnt_displacement_y} ${jnt_displacement_z}"
+                rpy="${jnt_rotation_x} ${jnt_rotation_y} ${jnt_rotation_z}" />
+            <parent link="${link_parent}" />
+            <child link="${camera_name}_Link" />
+            </joint>
+            <link name="${camera_name}_Link">
+            <visual>
+                <origin
+                xyz="${link_displacement_x} ${link_displacement_y} ${link_displacement_z}"
+                rpy="${link_rotation_x} ${link_rotation_y} ${link_rotation_z}" />
+                <geometry>
+                <cylinder length="0.01" radius="0.015" />
+                </geometry>
+                <material name="Blue" />
+            </visual>
+            <inertial>
+                <origin xyz="0 0 0" rpy="0 0 0" />
+                <mass value="1e-6" />
+                <inertia ixx="1e-12" ixy="0.0" ixz="0.0" iyy="1e-12" iyz="0.0"
+                izz="1e-12" />
+            </inertial>
+            </link>
+            <gazebo reference="${camera_name}_Link">
+                <sensor type="camera" name="${camera_name}">
+                    <update_rate>30.0</update_rate>
+                    <camera name="${camera_name}">
+                    <horizontal_fov>1.3962634</horizontal_fov>
+                    <image>
+                        <width>800</width>
+                        <height>800</height>
+                        <format>R8G8B8</format>
+                    </image>
+                    <clip>
+                        <near>0.1</near>
+                        <far>30</far>
+                    </clip>
+                    <noise>
+                        <type>gaussian</type>
+                        <!-- Noise is sampled independently per pixel on each frame. That pixel's
+                        noise value is added to each of its color channels, which at that point lie
+                        in the range [0,1]. -->
+                        <mean>0.0</mean>
+                        <stddev>0.007</stddev>
+                    </noise>
+                    </camera>
+                    <plugin name="camera_controller" filename="libgazebo_ros_camera.so">
+                    <alwaysOn>true</alwaysOn>
+                    <updateRate>0.0</updateRate>
+                    <cameraName>${camera_name}</cameraName>
+                    <imageTopicName>image_raw</imageTopicName>
+                    <cameraInfoTopicName>camera_info</cameraInfoTopicName>
+                    <frameName>${camera_name}_Link_frame</frameName>
+                    <hackBaseline>0.07</hackBaseline>
+                    <distortionK1>0.0</distortionK1>
+                    <distortionK2>0.0</distortionK2>
+                    <distortionK3>0.0</distortionK3>
+                    <distortionT1>0.0</distortionT1>
+                    <distortionT2>0.0</distortionT2>
+                    </plugin>
+                </sensor>
+            </gazebo>
+        </xacro:macro>
     </xacro:if>
     <xacro:macro name="sphere_inertia_def" params="radius mass">

File: nextagea_description/urdf/nextagea.urdf.xacro (robot description, xacro)
@@ -19,7 +19,8 @@
   <xacro:include filename="$(find nextagea_description)/urdf/base/nextagea_base.xacro" />
   <xacro:include filename="$(find nextagea_description)/urdf/robot/nextagea_robot.xacro" />
-  <xacro:include filename="$(find nextagea_description)/urdf/tool/nxao_gz_camera.xacro" />
+  <xacro:include filename="$(find nextagea_description)/urdf/tool/nextagea_tools.xacro" />
   <!-- Include files for extensions here -->
   <xacro:include filename="$(find nextage_extensions)/urdf/intel_realsense.xacro" />
+  <xacro:include filename="$(find nextage_extensions)/urdf/azure_kinect.xacro" />
   <xacro:include filename="$(find nextage_extensions)/urdf/imu.xacro" />
   <xacro:include filename="$(find nextage_extensions)/urdf/hexe.xacro" />
@@ -27,18 +28,37 @@
   <xacro:include filename="$(find nextage_extensions)/urdf/robotiq_85_gripper.xacro" />
   <xacro:include filename="$(find nextage_extensions)/urdf/robolimb.xacro" />
-  <xacro:include filename="$(find nextage_extensions)/urdf/kinect.xacro" />
   <!-- Include the nextagea base, robot torso, and tools -->
   <xacro:nextagea_robot/>
   <xacro:nextagea_base/>
-  <xacro:nextagea_tools use_hand_cameras="true" use_ft_sensors="true"/>
+  <xacro:nextagea_tools prefix="L" use_cables="true"/>
+  <xacro:nextagea_tools prefix="R" use_cables="false"/>
   <!-- Include files for extensions here -->
+  <xacro:property name="arm_tip" value="ARM_JOINT5_Link" />
+  <xacro:property name="arm_tip" value="ARM_ft_Link" />
   <!-- Sensors -->
-  <xacro:intel_realsense/>
-  <xacro:imu/>
-  <xacro:nx_kinect/>
-  <!-- <xacro:hex_e/> -->
+  <xacro:nx_intel_realsense_mount/>
+  <xacro:imu parent="base_link">
+    <origin xyz="0 0 0.3" rpy="0 0 0"/>
+  </xacro:imu>
+  <!-- Attach the HEX-E sensor  README -->
+  <xacro:property name="arm_tip" value="ARM_JOINT5_Link" />
+  <xacro:hex_e_ft_sensor prefix="LARM_" parent="L${arm_tip}" topic_name="ft_left/raw/data">
+    <origin xyz="0 0 0" rpy="0 0 0"/>
+  </xacro:hex_e_ft_sensor>
+  <xacro:hex_e_ft_sensor prefix="RARM_" parent="R${arm_tip}" topic_name="ft_right/raw/data">
+    <origin xyz="0 0 0" rpy="0 0 0"/>
+  </xacro:hex_e_ft_sensor>
+  <xacro:nx_kinect_mount/>
+  <!-- <xacro:nx_intel_realsense_azure_topics_mount/> -->
   <!-- Actuators -->
-  <!-- <xacro:robotiq_140/>
-  <xacro:robotiq_85/>
-  <xacro:robolimb/> -->
+  <xacro:property name="arm_tip" value="ARM_ft_Link" />
+  <xacro:robotiq_140_gripper prefix="left_" parent="L${arm_tip}">
+    <origin xyz="0 0 0" rpy="0 3.1415 0"/>
+  </xacro:robotiq_140_gripper>
+  <xacro:robotiq_85_gripper prefix="right_" parent="R${arm_tip}">
+      <origin xyz="0 0 0" rpy="0 3.1415 0"/>
+  </xacro:robotiq_85_gripper>
+  <!-- <xacro:robolimb_attach prefix="right" parent="R${arm_tip}">
+    <origin xyz="0 0 -0.12" rpy="3.14 0 -1.57"/>
+  </xacro:robolimb_attach> -->
 </robot>

File: nextagea_description/urdf/robot/nextagea_robot.xacro (robot description, xacro)
@@ -4,4 +4,19 @@
   <!-- nextagea robot macro -->
   <xacro:macro name="nextagea_robot" params="namespace:=/nextagea/ nextagea_gazebo_ros_control:=true">
+    <!-- NOTE: The poses of headmount and hand cameras are NOT precisely adjusted to
+    the 3D model nor the actual hardware config. These configs
+    are meant for a rapid prototyping only. -->
+    <xacro:camera_joint_link_gzplugin
+        camera_name="CAMERA_HEAD_L" link_parent="HEAD_JOINT1_Link"
+        jnt_displacement_x="${jnt_head_camera_displacement_x}" jnt_displacement_y="${jnt_head_camera_displacement_y}" jnt_displacement_z="${jnt_head_camera_displacement_z}"
+        jnt_rotation_x="0" jnt_rotation_y="${jnt_head_camera_rot_y}" jnt_rotation_z="0"
+        link_displacement_x="0.0325" link_displacement_y="0" link_displacement_z="0"
+        link_rotation_x="0" link_rotation_y="${M_PI/2}" link_rotation_z="-${link_head_camera_rot_z}" />
+    <xacro:camera_joint_link_gzplugin
+        camera_name="CAMERA_HEAD_R" link_parent="HEAD_JOINT1_Link"
+        jnt_displacement_x="${jnt_head_camera_displacement_x}" jnt_displacement_y="-${jnt_head_camera_displacement_y}" jnt_displacement_z="${jnt_head_camera_displacement_z}"
+        jnt_rotation_x="0" jnt_rotation_y="${jnt_head_camera_rot_y}" jnt_rotation_z="0"
+        link_displacement_x="0.0325" link_displacement_y="0" link_displacement_z="0"
+        link_rotation_x="0" link_rotation_y="${M_PI/2}" link_rotation_z="${link_head_camera_rot_z}" />
     <xacro:gazebo_nx_link name="WAIST" color="Black" />
     <link name="WAIST">

Commit message: Remove hardwareInterface from actuator

File: nextagea_description/urdf/general/common.xacro (robot description, xacro)
@@ -16,12 +16,11 @@
         <xacro:macro name="transmission_nx_joint" params="name">
             <transmission name="${name}_Trans">
-            <type>transmission_interface/SimpleTransmission</type>
-            <joint name="${name}">
-                <hardwareInterface>hardware_interface/PositionJointInterface</hardwareInterface>
-            </joint>
-            <actuator name="${name}_Motor">
-                <hardwareInterface>hardware_interface/PositionJointInterface</hardwareInterface>
-                <mechanicalReduction>1</mechanicalReduction>
-            </actuator>
+                <type>transmission_interface/SimpleTransmission</type>
+                <joint name="${name}">
+                    <hardwareInterface>hardware_interface/PositionJointInterface</hardwareInterface>
+                </joint>
+                <actuator name="${name}_Motor">
+                    <mechanicalReduction>1</mechanicalReduction>
+                </actuator>
             </transmission>
         </xacro:macro>
